File: Brains.kicad_sch (KiCad schematic)
At the start: 49 parts, among them J1 Conn_01x02_Pin, J3 USB_B_Micro, SW1 SW_SPST, SW2 SW_SPST, U1 ESP32-S3-WROOM-1, U2 LM78M05_TO220, U3 AMS1117-3.3, U5 USBLC6-2SC6, U6 W25Q16JVSS

Commit message: Changed LDO to AP2112K-3.3, Updated Layout
Parts:
- removed U3: AMS1117-3.3, Package_TO_SOT_SMD:SOT-223-3_TabPin2, symbol Regulator_Linear:AMS1117-3.3
- added U7: AP2112K-3.3, Package_TO_SOT_SMD:SOT-23-5, symbol Regulator_Linear:AP2112K-3.3
- C1, C3, C5, C8: value tbd -> 10uF
- C2, C4, C6, C7: value tbd -> 1uF
Connections:
- net +3.3V: now also U7.5 (VOUT)
- net 5Vin: now also U7.1 (VIN), U7.3 (EN)
- net GND: now also U7.2 (GND)
